Commit message: added xml tags; added xacro version

File: robots/wsg_32_description.urdf.xacro (robot description, xacro)
@@ -1,7 +1,12 @@
 <?xml version="1.0"?>
-<robot
-  name="wsg_32_description">
-  <link
-    name="hand_link">
+<robot xmlns:xacro="http://ros.org/wiki/xacro"  name="wsg_32_description">
+<xacro:macro name="wsg_32_xacro" params="name parent *origin">
+  <joint name="${name}_base_joint" type="fixed">
+    <insert_block name="origin"/>
+    <parent link="${parent}"/>
+    <child link="${name}_hand_link"/>
+  </joint>
+  <link
+    name="${name}_hand_link">
     <inertial>
       <origin
@@ -43,5 +48,5 @@
   </link>
   <link
-    name="left_finger_link">
+    name="${name}_left_finger_link">
     <inertial>
       <origin
@@ -83,13 +88,11 @@
   </link>
   <joint
-    name="left_finger_joint"
+    name="${name}_left_finger_joint"
     type="prismatic">
     <origin
       xyz="-0.0003903 -0.0358 0.069014"
       rpy="3.1416 -1.5708 0" />
-    <parent
-      link="hand_link" />
-    <child
-      link="left_finger_link" />
+    <parent link="${name}_hand_link" />
+    <child link="${name}_left_finger_link" />
     <axis
       xyz="0 1 0" />
@@ -101,5 +104,5 @@
   </joint>
   <link
-    name="right_finger_link">
+    name="${name}_right_finger_link">
     <inertial>
       <origin
@@ -141,13 +144,11 @@
   </link>
   <joint
-    name="right_finger_joint"
+    name="${name}_right_finger_joint"
     type="prismatic">
     <origin
       xyz="-0.0003903 0.0358 0.069012"
       rpy="1.5708 -1.5708 0" />
-    <parent
-      link="hand_link" />
-    <child
-      link="right_finger_link" />
+    <parent link="${name}_hand_link" />
+    <child link="${name}_right_finger_link" />
     <axis
       xyz="0 0 -1" />
@@ -160,5 +161,5 @@
   <!-- add fingers to actuated segments -->
   <link
-    name="right_universal_finger_link">
+    name="${name}_right_universal_finger_link">
     <inertial>
       <origin
@@ -200,16 +201,14 @@
   </link>
   <joint
-    name="right_universal_finger_joint"
+    name="${name}_right_universal_finger_joint"
     type="fixed">
     <origin
       xyz="0.00755 0.0 0.0049"
       rpy="0 1.57079 -1.57079" />
-    <parent
-      link="right_finger_link" />
-    <child
-      link="right_universal_finger_link" />
-  </joint>
-  <link
-    name="left_universal_finger_link">
+    <parent link="${name}_right_finger_link" />
+    <child link="${name}_right_universal_finger_link" />
+  </joint>
+  <link
+    name="${name}_left_universal_finger_link">
     <inertial>
       <origin
@@ -251,13 +250,12 @@
   </link>
   <joint
-    name="left_universal_finger_joint"
+    name="${name}_left_universal_finger_joint"
     type="fixed">
     <origin
       xyz="0.00755 -0.0045 0"
       rpy="0 3.14159 -1.57079" />
-    <parent
-      link="left_finger_link" />
-    <child
-      link="left_universal_finger_link" />
-  </joint>
+    <parent link="${name}_left_finger_link" />
+    <child link="${name}_left_universal_finger_link" />
+  </joint>
+</xacro:macro>
 </robot>
