Commit message: changed link names to match that of the wsg_50 ros driver

File: robots/wsg_32_description.URDF (robot description, URDF)
Before this commit: robot wsg_32_description, 5 links, 4 joints
Links:
- removed link left_finger_link
- removed link right_finger_link
- added link wsg_50_gripper_base_link_gripper_left, mass 3.41920163633724E-06; collision mesh filename=package://wsg_32_description/meshes/left_finger_link.STL; visual mesh filename=package://wsg_32_description/meshes/left_finger_link.STL
- added link wsg_50_gripper_base_link_gripper_right, mass 3.41920163633724E-06; collision mesh filename=package://wsg_32_description/meshes/right_finger_link.STL; visual mesh filename=package://wsg_32_description/meshes/right_finger_link.STL
Joints:
- removed joint left_finger_joint
- removed joint right_finger_joint
- added joint wsg_50_gripper_base_joint_gripper_left: type prismatic, parent hand_link, child wsg_50_gripper_base_link_gripper_left, origin xyz=-0.0003903 -0.0358 0.069014 rpy=3.1416 -1.5708 0, axis 0 1 0, limit lower=-0.028 upper=0 effort=0 velocity=0
- added joint wsg_50_gripper_base_joint_gripper_right: type prismatic, parent hand_link, child wsg_50_gripper_base_link_gripper_right, origin xyz=-0.0003903 0.0358 0.069012 rpy=1.5708 -1.5708 0, axis 0 0 -1, limit lower=-0.028 upper=0 effort=0 velocity=0
- joint left_universal_finger_joint: parent left_finger_link -> wsg_50_gripper_base_link_gripper_left
- joint right_universal_finger_joint: parent right_finger_link -> wsg_50_gripper_base_link_gripper_right

File: robots/wsg_32_description.urdf.xacro (robot description, xacro)
@@ -5,8 +5,8 @@
     <insert_block name="origin"/>
     <parent link="${parent}"/>
-    <child link="${name}_hand_link"/>
-  </joint>
-  <link
-    name="${name}_hand_link">
+    <child link="${name}_base_link"/>
+  </joint>
+  <link
+    name="${name}_base_link">
     <inertial>
       <origin
@@ -48,5 +48,5 @@
   </link>
   <link
-    name="${name}_left_finger_link">
+    name="${name}_base_link_gripper_left">
     <inertial>
       <origin
@@ -88,11 +88,11 @@
   </link>
   <joint
-    name="${name}_left_finger_joint"
+    name="${name}_base_joint_gripper_left"
     type="prismatic">
     <origin
       xyz="-0.0003903 -0.0358 0.069014"
       rpy="3.1416 -1.5708 0" />
-    <parent link="${name}_hand_link" />
-    <child link="${name}_left_finger_link" />
+    <parent link="${name}_base_link" />
+    <child link="${name}_base_link_gripper_left" />
     <axis
       xyz="0 1 0" />
@@ -104,5 +104,5 @@
   </joint>
   <link
-    name="${name}_right_finger_link">
+    name="${name}_base_link_gripper_right">
     <inertial>
       <origin
@@ -144,11 +144,11 @@
   </link>
   <joint
-    name="${name}_right_finger_joint"
+    name="${name}_base_joint_gripper_right"
     type="prismatic">
     <origin
       xyz="-0.0003903 0.0358 0.069012"
       rpy="1.5708 -1.5708 0" />
-    <parent link="${name}_hand_link" />
-    <child link="${name}_right_finger_link" />
+    <parent link="${name}_base_link" />
+    <child link="${name}_base_link_gripper_right" />
     <axis
       xyz="0 0 -1" />
@@ -206,5 +206,5 @@
       xyz="0.00755 0.0 0.0049"
       rpy="0 1.57079 -1.57079" />
-    <parent link="${name}_right_finger_link" />
+    <parent link="${name}_base_link_gripper_right" />
     <child link="${name}_right_universal_finger_link" />
   </joint>
@@ -255,5 +255,5 @@
       xyz="0.00755 -0.0045 0"
       rpy="0 3.14159 -1.57079" />
-    <parent link="${name}_left_finger_link" />
+    <parent link="${name}_base_link_gripper_left" />
     <child link="${name}_left_universal_finger_link" />
   </joint>

Commit message: modified fingers to accurately model the movement and jointstate of the wsg driver

File: robots/wsg_32_description.URDF (robot description, URDF)
Before this commit: robot wsg_32_description, 5 links, 4 joints
Joints:
- joint right_universal_finger_joint: origin xyz=0.00755 0.0 0.0049 rpy=0 1.57079 -1.57079 -> xyz=0.00755 0.0 0.0049 rpy=0 -1.57079 -1.57079
- joint wsg_50_gripper_base_joint_gripper_left: axis 0 1 0 -> 0 -1 0; origin xyz=-0.0003903 -0.0358 0.069014 rpy=3.1416 -1.5708 0 -> xyz=-0.0003903 -0.0078 0.069014 rpy=3.1416 -1.5708 0
- joint wsg_50_gripper_base_joint_gripper_right: axis 0 0 -1 -> 0 0 1; limit lower=-0.028 upper=0 effort=0 velocity=0 -> lower=0 upper=0.028 effort=0 velocity=0; origin xyz=-0.0003903 0.0358 0.069012 rpy=1.5708 -1.5708 0 -> xyz=-0.0003903 0.0078 0.069012 rpy=-1.5708 -1.5708 0

File: robots/wsg_32_description.urdf.xacro (robot description, xacro)
@@ -91,10 +91,10 @@
     type="prismatic">
     <origin
-      xyz="-0.0003903 -0.0358 0.069014"
+      xyz="-0.0003903 -0.0078 0.069014"
       rpy="3.1416 -1.5708 0" />
     <parent link="${name}_base_link" />
     <child link="${name}_base_link_gripper_left" />
     <axis
-      xyz="0 1 0" />
+      xyz="0 -1 0" />
     <limit
       lower="-0.028"
@@ -108,5 +108,5 @@
       <origin
         xyz="-2.72000777333109E-05 -0.00460993992652343 -0.00191114282807962"
-        rpy="0 0 0" />
+        rpy="-1.57079 3.14159 -1.57079" />
       <mass
         value="3.41920163633724E-06" />
@@ -122,5 +122,5 @@
       <origin
         xyz="-0.00725 0 0.0004"
-        rpy="-1.57079 0  -1.57079" />
+        rpy="-1.57079 3.14159  -1.57079" />
       <geometry>
         <mesh
@@ -147,13 +147,13 @@
     type="prismatic">
     <origin
-      xyz="-0.0003903 0.0358 0.069012"
-      rpy="1.5708 -1.5708 0" />
+      xyz="-0.0003903 0.0078 0.069012"
+      rpy="-1.5708 -1.5708 0" />
     <parent link="${name}_base_link" />
     <child link="${name}_base_link_gripper_right" />
     <axis
-      xyz="0 0 -1" />
+      xyz="0 0 1" />
     <limit
-      lower="-0.028"
-      upper="0"
+      lower="0"
+      upper="0.028"
       effort="0"
       velocity="0" />
@@ -178,5 +178,5 @@
     <visual>
       <origin
-        xyz="-0.00 0 0.00"
+        xyz="-0.01 0 0.00"
         rpy="0 0 0" />
       <geometry>
@@ -205,5 +205,5 @@
     <origin
       xyz="0.00755 0.0 0.0049"
-      rpy="0 1.57079 -1.57079" />
+      rpy="0 -1.57079 -1.57079" />
     <parent link="${name}_base_link_gripper_right" />
     <child link="${name}_right_universal_finger_link" />
